File: hardware/ACNode-Shield/ACNode-Shield-2x2.kicad_pcb (KiCad board)
At the start: 2 copper layers, 110 x 110 mm, 64 parts, among them J111111 MICRO_SD_HINGE, J111112 MICRO_SD_HINGE, J111121 MICRO_SD_HINGE, J111122 MICRO_SD_HINGE, P111111 CONN_NFC, P111111 CONN_RELAY, P111111 CONN_RGB_LED, P111111 CONN_WS2812, P111111 CONN_X6, P111111 CONN_X7, P111112 CONN_NFC, P111112 CONN_RELAY, P111112 CONN_RGB_LED, P111112 CONN_WS2812, P111112 CONN_X6, P111112 CONN_X7, P111121 CONN_NFC, P111121 CONN_RELAY, P111121 CONN_RGB_LED, P111121 CONN_WS2812, P111121 CONN_X6, P111121 CONN_X7, P111122 CONN_NFC, P111122 CONN_RELAY, P111122 CONN_RGB_LED, P111122 CONN_WS2812, P111122 CONN_X6, P111122 CONN_X7, Q111111 PN2222A, Q111112 PN2222A, Q111121 PN2222A, Q111122 PN2222A, SW111111 SW_BTN, SW111111 SW_RST, SW111112 SW_BTN, SW111112 SW_RST, SW111121 SW_BTN, SW111121 SW_RST, SW111122 SW_BTN, SW111122 SW_RST, U111111 SRD-05VDC-SL-C, U111111 WS2812B, U111112 SRD-05VDC-SL-C, U111112 WS2812B, U111121 SRD-05VDC-SL-C, U111121 WS2812B, U111122 SRD-05VDC-SL-C, U111122 WS2812B

Commit message: Generated 2x2 board matrix.
Parts:
- removed C111111, C111112, C111121, C111122: 10nF, Capacitors_SMD:C_1210_HandSoldering
- removed D111112, D111121, D111122: 1N4007, Diodes_ThroughHole:Diode_DO-41_SOD81_Horizontal_RM10
- removed J111111, J111112, J111121, J111122: MICRO_SD_HINGE, armory:MICRO_SD_HINGE_AMP
- removed P111112, P111121, P111122: CONN_RELAY, Pin_Headers:Pin_Header_Straight_1x03
- removed P111112, P111121, P111122: CONN_RGB_LED, Pin_Headers:Pin_Header_Straight_1x04
- removed P111112, P111121, P111122: CONN_WS2812, Pin_Headers:Pin_Header_Straight_1x03
- removed P111112, P111121, P111122: CONN_NFC, Pin_Headers:Pin_Header_Straight_1x04
- removed P111112, P111121, P111122: CONN_X7, Socket_Strips:Socket_Strip_Straight_2x10
- removed P111112, P111121, P111122: CONN_X6, Socket_Strips:Socket_Strip_Straight_2x10
- removed Q111112, Q111121, Q111122: PN2222A, TO_SOT_Packages_THT:TO-92_Inline_Wide
- removed R111111, R111112, R111121, R111122: 100, Resistors_ThroughHole:Resistor_Horizontal_RM10mm
- removed R111112, R111121, R111122: 10k, Resistors_ThroughHole:Resistor_Horizontal_RM10mm
- removed SW111112, SW111121, SW111122: SW_RST, Buttons_Switches_ThroughHole:SW_PUSH_SMALL
- removed SW111112, SW111121, SW111122: SW_BTN, Socket_Strips:Socket_Strip_Straight_1x02
- removed U111112, U111121, U111122: SRD-05VDC-SL-C, Relays_ThroughHole:Relay_SANYOU_SRD_Series_Form_C
- removed U111112, U111121, U111122: WS2812B, ws2812:WS2812b
- added C11: C_Small, Capacitors_SMD:C_1206, B.Cu at (48.0, 38.1)
- added C12: C_Small, Capacitors_SMD:C_1206, B.Cu at (48.0, 98.1)
- added C21: C_Small, Capacitors_SMD:C_1206, B.Cu at (108.0, 38.1)
- added C22: C_Small, Capacitors_SMD:C_1206, B.Cu at (108.0, 98.1)
- added D12: 1N4007, Diodes_ThroughHole:Diode_DO-41_SOD81_Horizontal_RM10, F.Cu at (48.7, 114.6)
- added D21: 1N4007, Diodes_ThroughHole:Diode_DO-41_SOD81_Horizontal_RM10, F.Cu at (108.7, 54.6)
- added D22: 1N4007, Diodes_ThroughHole:Diode_DO-41_SOD81_Horizontal_RM10, F.Cu at (108.7, 114.6)
- added J11: MICRO_SD_HINGE, MicroSD:MICRO_SD_HINGE_CHINA, F.Cu at (46.7, 23.4)
- added J12: MICRO_SD_HINGE, MicroSD:MICRO_SD_HINGE_CHINA, F.Cu at (46.7, 83.4)
- added J21: MICRO_SD_HINGE, MicroSD:MICRO_SD_HINGE_CHINA, F.Cu at (106.7, 23.4)
- added J22: MICRO_SD_HINGE, MicroSD:MICRO_SD_HINGE_CHINA, F.Cu at (106.7, 83.4)
- added P12: CONN_RELAY, Pin_Headers:Pin_Header_Straight_1x03, B.Cu at (22.5, 118.2)
- added P12: CONN_RGB_LED, Pin_Headers:Pin_Header_Straight_1x04, B.Cu at (27.5, 94.8)
- added P12: CONN_WS2812, Pin_Headers:Pin_Header_Straight_1x03, B.Cu at (34.0, 86.5)
- added P12: CONN_NFC, Pin_Headers:Pin_Header_Straight_1x04, B.Cu at (49.2, 105.2)
- added P12: CONN_X7, Socket_Strips:Socket_Strip_Straight_2x10, F.Cu at (23.6, 87.4)
- added P12: CONN_X6, Socket_Strips:Socket_Strip_Straight_2x10, F.Cu at (66.8, 87.4)
- added P21: CONN_RELAY, Pin_Headers:Pin_Header_Straight_1x03, B.Cu at (82.5, 58.2)
- added P21: CONN_RGB_LED, Pin_Headers:Pin_Header_Straight_1x04, B.Cu at (87.5, 34.8)
- added P21: CONN_WS2812, Pin_Headers:Pin_Header_Straight_1x03, B.Cu at (94.0, 26.5)
- added P21: CONN_NFC, Pin_Headers:Pin_Header_Straight_1x04, B.Cu at (109.2, 45.2)
- added P21: CONN_X7, Socket_Strips:Socket_Strip_Straight_2x10, F.Cu at (83.6, 27.4)
- added P21: CONN_X6, Socket_Strips:Socket_Strip_Straight_2x10, F.Cu at (126.8, 27.4)
- added P22: CONN_RELAY, Pin_Headers:Pin_Header_Straight_1x03, B.Cu at (82.5, 118.2)
- added P22: CONN_RGB_LED, Pin_Headers:Pin_Header_Straight_1x04, B.Cu at (87.5, 94.8)
- added P22: CONN_WS2812, Pin_Headers:Pin_Header_Straight_1x03, B.Cu at (94.0, 86.5)
- added P22: CONN_NFC, Pin_Headers:Pin_Header_Straight_1x04, B.Cu at (109.2, 105.2)
- added P22: CONN_X7, Socket_Strips:Socket_Strip_Straight_2x10, F.Cu at (83.6, 87.4)
- added P22: CONN_X6, Socket_Strips:Socket_Strip_Straight_2x10, F.Cu at (126.8, 87.4)
- added Q12: PN2222A, TO_SOT_Packages_THT:TO-92_Inline_Wide, F.Cu at (45.9, 105.2)
- added Q21: PN2222A, TO_SOT_Packages_THT:TO-92_Inline_Wide, F.Cu at (105.9, 45.2)
- added Q22: PN2222A, TO_SOT_Packages_THT:TO-92_Inline_Wide, F.Cu at (105.9, 105.2)
- added R12: 1k, Resistors_ThroughHole:Resistor_Horizontal_RM10mm, F.Cu at (41.1, 97.3)
- added R21: 1k, Resistors_ThroughHole:Resistor_Horizontal_RM10mm, F.Cu at (101.1, 37.3)
- added R22: 1k, Resistors_ThroughHole:Resistor_Horizontal_RM10mm, F.Cu at (101.1, 97.3)
- added SW12: SW_RST, Buttons_Switches_ThroughHole:SW_PUSH_SMALL, B.Cu at (34.5, 104.8)
- added SW12: SW_BTN, Socket_Strips:Socket_Strip_Straight_1x02, B.Cu at (21.2, 83.8)
- added SW21: SW_RST, Buttons_Switches_ThroughHole:SW_PUSH_SMALL, B.Cu at (94.5, 44.8)
- added SW21: SW_BTN, Socket_Strips:Socket_Strip_Straight_1x02, B.Cu at (81.2, 23.8)
- added SW22: SW_RST, Buttons_Switches_ThroughHole:SW_PUSH_SMALL, B.Cu at (94.5, 104.8)
- added SW22: SW_BTN, Socket_Strips:Socket_Strip_Straight_1x02, B.Cu at (81.2, 83.8)
- added U12: SRD-05VDC-SL-C, Relays_ThroughHole:Relay_SANYOU_SRD_Series_Form_C, B.Cu at (44.2, 119.5)
- added U12: WS2812B, ws2812:WS2812b, B.Cu at (56.7, 85.5)
- added U21: SRD-05VDC-SL-C, Relays_ThroughHole:Relay_SANYOU_SRD_Series_Form_C, B.Cu at (104.2, 59.5)
- added U21: WS2812B, ws2812:WS2812b, B.Cu at (116.7, 25.5)
- added U22: SRD-05VDC-SL-C, Relays_ThroughHole:Relay_SANYOU_SRD_Series_Form_C, B.Cu at (104.2, 119.5)
- added U22: WS2812B, ws2812:WS2812b, B.Cu at (116.7, 85.5)
- R11: renamed from R111111; value 10k -> 1k
- moved U11 28.8 mm to (56.7, 25.5), turned to 180 degrees
- moved P11 20.9 mm to (49.2, 45.2), turned to 270 degrees
- renumbered D111111 to D11, P111111 to P11, Q111111 to Q11, SW111111 to SW11, U111111 to U11
Connections:
- Q11 pad 1: Net-(Q1-Pad1) -> GND
Routing:
- net PP5: track 56.1 -> 147.4 mm
- net (no net): track 128.0 -> 64.0 mm
- net Net-(P6-Pad2): track 38.7 -> 101.2 mm
- net PQ0: track 165.6 -> 109.5 mm
- net PP0: track 30.4 -> 78.6 mm
- net +3.3v: track 225.5 -> 271.9 mm
- net PQ3: track 146.6 -> 189.4 mm
- net PQ2: track 196.2 -> 162.7 mm
- net PP1: track 30.5 -> 63.8 mm
- net Net-(Q1-Pad1): track 25.9 -> 0.00 mm
- net +5V: track 402.0 -> 426.7 mm
- net PQ1: track 107.6 -> 128.3 mm
- net /RESET: track 65.0 -> 72.5 mm
- net Net-(D1-Pad2): track 121.8 -> 114.3 mm
- net GND: track 433.6 -> 436.3 mm
Other:
- net class +3.3v added: clearance 0.2, trace_width 0.5, via_dia 0.6, via_drill 0.4
- net class +5V added: clearance 0.2, trace_width 0.5, via_dia 0.6, via_drill 0.4
- net class GND added: clearance 0.2, trace_width 0.5, via_dia 0.6, via_drill 0.4
