File: hardware/New-New-ACNode-Shield/New-New-ACNode-Shield.kicad_pcb (KiCad board)
At the start: 2 copper layers, 55.9 x 124.5 mm, 48 parts, among them J1 8P8C_Shielded, J2 8P8C_Shielded, J3 Conn_01x02, J4 Conn_01x03, J5 Conn_01x02, J6 Conn_01x04_Female, J7 Conn_01x02, K1 SANYOU_SRD_Form_C, Q1 2N7002, Q2 2N7002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

Commit message: Slightly reworked New-New-ACNode-Shield
The ethernet connector was fouling the PCB, so this
is an attempt to create a suitable cutout. It involves moving the tool running detection.
Parts:
- added J8: Conn_01x03, Connector_PinHeader_2.54mm:PinHeader_1x03_P2.54mm_Vertical, F.Cu at (156.7, 88.7)
- moved J5 46.0 mm to (174.3, 162.5), turned to 90 degrees
- moved R11 32.4 mm to (167.6, 164.9), turned to 0 degrees
- moved U4 22.0 mm to (161.7, 161.7), turned to 270 degrees
- moved J4 1.75 mm to (127.3, 145.1)
- moved K1 1.46 mm to (154.9, 145.1)
Connections:
- U1 pad 3: GND -> Net-(J8-Pad2)
Routing:
- net /~ToolOn: track 184.9 -> 167.0 mm
- net Net-(J8-Pad2): track 0.00 -> 8.72 mm, vias 0 -> 1
- net /Reader_SerialTx: track 100.5 -> 106.2 mm
- net +3V3: track 219.4 -> 223.5 mm
- net GND: track 34.5 -> 31.6 mm, vias 30 -> 29
- net Net-(R11-Pad1): track 2.00 -> 3.47 mm
- net Net-(J5-Pad2): track 5.05 -> 6.02 mm
- net Net-(J5-Pad1): track 3.59 -> 2.72 mm
- net /Reader_SerialRx: track 92.5 -> 93.3 mm
- net /LED_G_Trigger: track 86.2 -> 86.9 mm
- net /LED_B_Trigger: track 94.5 -> 95.2 mm
- net +5V: track 120.2 -> 120.8 mm
- net Net-(D2-Pad2): track 14.0 -> 14.6 mm
Other:
- outline, holes or cut-outs redrawn
- board text added: "ACNode New New Shield Aug 2021 Michael Cullen"
- board text removed: "ACNode New New Shield Feb 2021 Michael Cullen"
